File: Macintosh II Video Breakout/Macintosh II Video Breakout.sch (KiCad schematic (older format))
At the start: 12 parts, among them J1 RED, J2 BlU, J3 GRN, J4 VSYNC, J5 CSYNC, J6 HSYNC, J7 DB15_Male, J8 DB15_Female

Commit message: PCB
Connections:
- net BLU.GND is gone; now on net GND: J2.2 (Ext), J7.13 (P13), J8.13 (P13)
- net C&VSYNC.GND is gone; now on net GND: J4.2 (Ext), J5.2 (Ext), J7.11 (P111), J8.11 (P111)
- net GRN.GND is gone; now on net GND: J3.2 (Ext), J7.6, J8.6
- net HSYNC.GND is gone; now on net GND: J6.2 (Ext), J7.14 (P14), J8.14 (P14)
- net RED.GND is gone; now on net GND: J1.2 (Ext), J7.1, J8.1
Changed lines of the file:
@@
 $EndComp
 Text GLabel 5050 4600 0    50   Output ~ 0
-RED.GND
+GND
 Text GLabel 5050 4500 0    50   Output ~ 0
 BLU.VID
@@
 CSYNC
 Text GLabel 5050 4100 0    50   Output ~ 0
-C&VSYNC.GND
+GND
 Text GLabel 5050 4000 0    50   Output ~ 0
 SENSE0
@@
 GRN.VID
 Text GLabel 5050 3700 0    50   Output ~ 0
-BLU.GND
+GND
 Text GLabel 5050 3600 0    50   Output ~ 0
-GRN.GND
+GND
 Text GLabel 5050 3500 0    50   Output ~ 0
-HSYNC.GND
+GND
 Text GLabel 5050 3400 0    50   Output ~ 0
 SENSE1
@@
 HSYNC
 Text GLabel 6700 3200 0    50   Input ~ 0
-RED.GND
+GND
 Text GLabel 6700 3300 0    50   Input ~ 0
 BLU.VID
@@
 CSYNC
 Text GLabel 6700 3700 0    50   Input ~ 0
-C&VSYNC.GND
+GND
 Text GLabel 6700 3800 0    50   Input ~ 0
 SENSE0
@@
 GRN.VID
 Text GLabel 6700 4100 0    50   Input ~ 0
-BLU.GND
+GND
 Text GLabel 6700 4200 0    50   Input ~ 0
-GRN.GND
+GND
 Text GLabel 6700 4300 0    50   Input ~ 0
-HSYNC.GND
+GND
 Text GLabel 6700 4400 0    50   Input ~ 0
 SENSE1
@@
 RED.VID
 Text GLabel 4700 1050 0    50   Input ~ 0
-RED.GND
+GND
 $Comp
 L Connector:Conn_Coaxial J2
@@
 BLU.VID
 Text GLabel 4700 1600 0    50   Input ~ 0
-BLU.GND
+GND
 Wire Wire Line
 	4700 1600 4900 1600
@@
 	4900 1600 4900 1500
 Text GLabel 4700 2150 0    50   Input ~ 0
-GRN.GND
+GND
 Text GLabel 4700 1850 0    50   Input ~ 0
 GRN.VID
@@
 VSYNC
 Text GLabel 5750 1050 0    50   Input ~ 0
-C&VSYNC.GND
+GND
 Text GLabel 5750 1600 0    50   Input ~ 0
-C&VSYNC.GND
+GND
 Text GLabel 5750 1300 0    50   Input ~ 0
 CSYNC
@@
 HSYNC
 Text GLabel 5750 2100 0    50   Input ~ 0
-HSYNC.GND
+GND
 Wire Wire Line
 	5950 2050 5950 2100
